File: audioModTC/audio.sch (KiCad schematic (older format))
At the start: 39 parts, among them J3 Audio-Jack-2, U10 LM2611A, U11 UCC37322P, U12 4N35, U6 AP3012, U7 LM741, U8 LM741, U9 LM741

Commit message: Finished PCB
Parts:
- added J4, J5: Conn_01x03, Pin_Headers:Pin_Header_Straight_1x03_Pitch2.54mm, symbol Conn_01x03
Connections:
- net +5V: now also J4.3 (Pin_3), J5.1 (Pin_1)
- net GNDA: now also J4.2 (Pin_2), J5.2 (Pin_2)
- net at R17.1: now also J4.1 (Pin_1); no longer U12.1
- new net: J5.3 (Pin_3), U12.1
Other:
- moved on the sheet: R18, U12
Changed lines of the file:
@@
 $EndComp
 $Comp
-L -15V #PWR19
+L -15V #PWR21
 U 1 1 5A4B51DD
 P 3675 2600
-F 0 "#PWR19" H 3675 2700 50  0001 C CNN
+F 0 "#PWR21" H 3675 2700 50  0001 C CNN
 F 1 "-15V" H 3675 2750 50  0000 C CNN
 F 2 "" H 3675 2600 50  0001 C CNN
@@
 $EndComp
 $Comp
-L -15V #PWR27
+L -15V #PWR29
 U 1 1 5A4B53F4
 P 4575 2675
-F 0 "#PWR27" H 4575 2775 50  0001 C CNN
+F 0 "#PWR29" H 4575 2775 50  0001 C CNN
 F 1 "-15V" H 4575 2825 50  0000 C CNN
 F 2 "" H 4575 2675 50  0001 C CNN
@@
 L 4N35 U12
 U 1 1 5A4BD550
-P 8200 2350
-F 0 "U12" H 8000 2550 50  0000 L CNN
-F 1 "4N35" H 8200 2550 50  0000 L CNN
-F 2 "Housings_DIP:DIP-6_W7.62mm" H 8000 2150 50  0001 L CIN
-F 3 "" H 8200 2250 50  0001 L CNN
-	1    8200 2350
+P 9100 2350
+F 0 "U12" H 8900 2550 50  0000 L CNN
+F 1 "4N35" H 9100 2550 50  0000 L CNN
+F 2 "Housings_DIP:DIP-6_W7.62mm" H 8900 2150 50  0001 L CIN
+F 3 "" H 9100 2250 50  0001 L CNN
+	1    9100 2350
 	1    0    0    -1
 $EndComp
@@
 L +5V #PWR025
 U 1 1 5A4BD5E0
-P 8500 2250
-F 0 "#PWR025" H 8500 2100 50  0001 C CNN
-F 1 "+5V" H 8500 2390 50  0000 C CNN
-F 2 "" H 8500 2250 50  0001 C CNN
-F 3 "" H 8500 2250 50  0001 C CNN
-	1    8500 2250
+P 9400 2250
+F 0 "#PWR025" H 9400 2100 50  0001 C CNN
+F 1 "+5V" H 9400 2390 50  0000 C CNN
+F 2 "" H 9400 2250 50  0001 C CNN
+F 3 "" H 9400 2250 50  0001 C CNN
+	1    9400 2250
 	1    0    0    -1
 $EndComp
@@
 L R R18
 U 1 1 5A4C0739
-P 8500 2750
-F 0 "R18" V 8580 2750 50  0000 C CNN
-F 1 "280" V 8500 2750 50  0000 C CNN
-F 2 "Resistors_SMD:R_0603" V 8430 2750 50  0001 C CNN
-F 3 "" H 8500 2750 50  0001 C CNN
-	1    8500 2750
-	1    0    0    -1
-$EndComp
-Wire Wire Line
-	8500 2600 8500 2450
-Text HLabel 8650 2450 2    60   Input ~ 0
+P 9400 2750
+F 0 "R18" V 9480 2750 50  0000 C CNN
+F 1 "280" V 9400 2750 50  0000 C CNN
+F 2 "Resistors_SMD:R_0603" V 9330 2750 50  0001 C CNN
+F 3 "" H 9400 2750 50  0001 C CNN
+	1    9400 2750
+	1    0    0    -1
+$EndComp
+Wire Wire Line
+	9400 2600 9400 2450
+Text HLabel 9550 2450 2    60   Input ~ 0
 Int
 Wire Wire Line
-	8500 2450 8650 2450
+	9400 2450 9550 2450
 $Comp
 L GND #PWR027
 U 1 1 5A4C09BC
-P 8500 2900
-F 0 "#PWR027" H 8500 2650 50  0001 C CNN
-F 1 "GND" H 8500 2750 50  0000 C CNN
-F 2 "" H 8500 2900 50  0001 C CNN
-F 3 "" H 8500 2900 50  0001 C CNN
-	1    8500 2900
+P 9400 2900
+F 0 "#PWR027" H 9400 2650 50  0001 C CNN
+F 1 "GND" H 9400 2750 50  0000 C CNN
+F 2 "" H 9400 2900 50  0001 C CNN
+F 3 "" H 9400 2900 50  0001 C CNN
+	1    9400 2900
 	1    0    0    -1
 $EndComp
@@
 $EndComp
 $Comp
-L -15V #PWR25
+L -15V #PWR27
 U 1 1 5A4C5AEF
 P 4125 4475
-F 0 "#PWR25" H 4125 4575 50  0001 C CNN
+F 0 "#PWR27" H 4125 4575 50  0001 C CNN
 F 1 "-15V" H 4125 4625 50  0000 C CNN
 F 2 "" H 4125 4475 50  0001 C CNN
@@
 Connection ~ 6800 6175
 $Comp
-L -15V #PWR37
+L -15V #PWR39
 U 1 1 5A4F2130
 P 7100 5300
-F 0 "#PWR37" H 7100 5400 50  0001 C CNN
+F 0 "#PWR39" H 7100 5400 50  0001 C CNN
 F 1 "-15V" H 7100 5450 50  0000 C CNN
 F 2 "" H 7100 5300 50  0001 C CNN
@@
 Wire Wire Line
 	2250 2250 2100 2250
+Wire Wire Line
+	7900 2300 7900 2250
+Wire Wire Line
+	7900 2400 7900 2450
+Wire Wire Line
+	8800 2300 8800 2250
+Wire Wire Line
+	8800 2400 8800 2450
+$Comp
+L GNDA #PWR039
+U 1 1 5A544CFD
+P 8950 2575
+F 0 "#PWR039" H 8950 2325 50  0001 C CNN
+F 1 "GNDA" H 8950 2425 50  0000 C CNN
+F 2 "" H 8950 2575 50  0001 C CNN
+F 3 "" H 8950 2575 50  0001 C CNN
+	1    8950 2575
+	1    0    0    -1
+$EndComp
+$Comp
+L Conn_01x03 J4
+U 1 1 5A54833A
+P 8100 2400
+F 0 "J4" H 8100 2600 50  0000 C CNN
+F 1 "Conn_01x03" H 8100 2200 50  0000 C CNN
+F 2 "Pin_Headers:Pin_Header_Straight_1x03_Pitch2.54mm" H 8100 2400 50  0001 C CNN
+F 3 "" H 8100 2400 50  0001 C CNN
+	1    8100 2400
+	1    0    0    -1
+$EndComp
+$Comp
+L Conn_01x03 J5
+U 1 1 5A5483D2
+P 8600 2400
+F 0 "J5" H 8600 2600 50  0000 C CNN
+F 1 "Conn_01x03" H 8600 2200 50  0000 C CNN
+F 2 "Pin_Headers:Pin_Header_Straight_1x03_Pitch2.54mm" H 8600 2400 50  0001 C CNN
+F 3 "" H 8600 2400 50  0001 C CNN
+	1    8600 2400
+	-1   0    0    1
+$EndComp
+Wire Wire Line
+	8800 2450 8850 2450
+Wire Wire Line
+	8850 2450 8850 2575
+Wire Wire Line
+	8850 2575 8950 2575
+$Comp
+L +5V #PWR040
+U 1 1 5A549EEB
+P 8750 2725
+F 0 "#PWR040" H 8750 2575 50  0001 C CNN
+F 1 "+5V" H 8750 2865 50  0000 C CNN
+F 2 "" H 8750 2725 50  0001 C CNN
+F 3 "" H 8750 2725 50  0001 C CNN
+	1    8750 2725
+	1    0    0    -1
+$EndComp
+$Comp
+L +5V #PWR041
+U 1 1 5A549F74
+P 7775 2700
+F 0 "#PWR041" H 7775 2550 50  0001 C CNN
+F 1 "+5V" H 7775 2840 50  0000 C CNN
+F 2 "" H 7775 2700 50  0001 C CNN
+F 3 "" H 7775 2700 50  0001 C CNN
+	1    7775 2700
+	1    0    0    -1
+$EndComp
+Wire Wire Line
+	7900 2700 7900 2500
+Wire Wire Line
+	8800 2725 8800 2500
+Wire Wire Line
+	8800 2725 8750 2725
+Wire Wire Line
+	7900 2700 7775 2700
 $EndSCHEMATC
