File: audioModTC/audioModTC.kicad_pcb (KiCad board)
At the start: 2 copper layers, 75 parts, among them J1 Screw_Terminal_01x02, J2 703W-00/52, J3 Audio-Jack-2, Q1 IRFP360LCPBF, Q2 IRFP360LCPBF, T1 Transformer_1P_2S, T2 Transformer_1P_1S, U1 NCP1117-12V, U10 LM2611A, U11 UCC37322P, U12 4N35, U2 74HC14, U3 NCP1117-5V, U4 UCC37321P, U5 UCC37322P, U6 AP3012, U7 LM741, U8 LM741, U9 LM741

Commit message: Finished PCB
Parts:
- added J4: Conn_01x03, Pin_Headers:Pin_Header_Straight_1x03_Pitch2.54mm, F.Cu at (101.7, 68.6)
- added J5: Conn_01x03, Pin_Headers:Pin_Header_Straight_1x03_Pitch2.54mm, F.Cu at (193.7, 67.9)
- C10, C11: footprint Capacitors_THT:CP_Radial_D6.3mm_P2.50mm -> Capacitors_THT:CP_Radial_D25.0mm_P10.00mm_SnapIn
- C12, C13: footprint Capacitors_SMD:C_0603 -> Capacitors_THT:C_Rect_L26.5mm_W7.0mm_P22.50mm_MKS4
- C2, C4, C6: value 100nF -> .1uF
- moved R18 118.2 mm to (170.8, 75.6), turned to 90 degrees
- moved R7 112.2 mm to (93.3, 83.8), turned to 180 degrees
- moved L11 94.9 mm to (101.7, 92.7)
- moved R8 94.2 mm to (99.2, 111.5), turned to 90 degrees
- moved L12 91.6 mm to (99.9, 88.9), turned to 180 degrees
- moved R17 91.3 mm to (101.7, 72.6), turned to 270 degrees
- moved C4 90.5 mm to (210.3, 81.0)
- moved C21 86.4 mm to (99.2, 86.9)
- moved R6 84.5 mm to (89.3, 84.8), turned to 90 degrees
- moved R16 83.7 mm to (104.5, 88.1), turned to 270 degrees
- moved D7 81.7 mm to (93.9, 97.0), turned to 270 degrees
- moved C2 80.2 mm to (190.0, 74.4), turned to 90 degrees
- moved U2 76.2 mm to (180.6, 124.5), turned to 90 degrees
- moved C20 75.4 mm to (102.2, 85.9), turned to 180 degrees
- moved U9 74.7 mm to (99.4, 130.5), turned to 90 degrees
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Connections:
- R17 pad 1: Net-(R17-Pad1) -> Net-(J4-Pad1)
- U12 pad 1: Net-(R17-Pad1) -> Net-(J5-Pad3)
Routing:
- net GNDA: track 0.00 -> 155.3 mm, vias 0 -> 11
- net Net-(C10-Pad2): track 0.00 -> 151.5 mm, vias 0 -> 1
- net Net-(C10-Pad1): track 0.00 -> 121.6 mm
- net +12V: track 0.00 -> 112.8 mm, vias 0 -> 2
- net +15V: track 0.00 -> 106.8 mm, vias 0 -> 1
- net Net-(D4-Pad2): track 0.00 -> 106.5 mm
- net Net-(Q1-Pad2): track 0.00 -> 95.7 mm, vias 0 -> 2
- net Net-(10k1-Pad3): track 0.00 -> 79.7 mm
- net /INT: track 0.00 -> 78.0 mm, vias 0 -> 2
- net GND: track 0.00 -> 74.1 mm, vias 0 -> 4
- net Net-(Q2-Pad2): track 0.00 -> 64.2 mm, vias 0 -> 3
- net -15V: track 0.00 -> 63.7 mm, vias 0 -> 3
- net +5V: track 0.00 -> 58.5 mm, vias 0 -> 2
- net Net-(D10-Pad1): track 0.00 -> 56.9 mm, vias 0 -> 2
- net Net-(R2-Pad1): track 0.00 -> 41.0 mm, vias 0 -> 2
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- added copper zone on F.Cu, net +5V
- added copper zone on B.Cu, net GND
- added copper zone on B.Cu, net GNDA
Other:
- board outline added: 137.2 x 66 mm

Commit message: Sent to fab house
Parts:
- added REF**: MouseBite, Custom:MouseBite, F.Cu at (109.2, 127.7)
- added REF**: MouseBite, Custom:MouseBite, F.Cu at (109.2, 118.7)
- added REF**: MouseBite, Custom:MouseBite, F.Cu at (109.2, 117.7)
- added REF**: MouseBite, Custom:MouseBite, F.Cu at (109.2, 116.7)
- added REF**: MouseBite, Custom:MouseBite, F.Cu at (109.2, 115.7)
- added REF**: MouseBite, Custom:MouseBite, F.Cu at (109.2, 114.7)
- added REF**: MouseBite, Custom:MouseBite, F.Cu at (109.2, 113.7)
- added REF**: MouseBite, Custom:MouseBite, F.Cu at (109.2, 112.7)
- added REF**: MouseBite, Custom:MouseBite, F.Cu at (109.2, 111.7)
- added REF**: MouseBite, Custom:MouseBite, F.Cu at (109.2, 110.7)
- added REF**: MouseBite, Custom:MouseBite, F.Cu at (109.2, 109.7)
- added REF**: MouseBite, Custom:MouseBite, F.Cu at (109.2, 126.7)
- added REF**: MouseBite, Custom:MouseBite, F.Cu at (109.2, 108.7)
- added REF**: MouseBite, Custom:MouseBite, F.Cu at (109.2, 107.7)
- added REF**: MouseBite, Custom:MouseBite, F.Cu at (109.2, 106.7)
- added REF**: MouseBite, Custom:MouseBite, F.Cu at (109.2, 105.7)
- added REF**: MouseBite, Custom:MouseBite, F.Cu at (109.2, 104.7)
- added REF**: MouseBite, Custom:MouseBite, F.Cu at (109.2, 103.7)
- added REF**: MouseBite, Custom:MouseBite, F.Cu at (109.2, 102.7)
- added REF**: MouseBite, Custom:MouseBite, F.Cu at (109.2, 101.7)
- added REF**: MouseBite, Custom:MouseBite, F.Cu at (109.2, 100.7)
- added REF**: MouseBite, Custom:MouseBite, F.Cu at (109.2, 99.7)
- added REF**: MouseBite, Custom:MouseBite, F.Cu at (109.2, 125.7)
- added REF**: MouseBite, Custom:MouseBite, F.Cu at (109.2, 98.7)
- added REF**: MouseBite, Custom:MouseBite, F.Cu at (109.2, 97.7)
- added REF**: MouseBite, Custom:MouseBite, F.Cu at (109.2, 96.7)
- added REF**: MouseBite, Custom:MouseBite, F.Cu at (109.2, 95.7)
- added REF**: MouseBite, Custom:MouseBite, F.Cu at (109.2, 94.7)
- added REF**: MouseBite, Custom:MouseBite, F.Cu at (109.2, 93.7)
- added REF**: MouseBite, Custom:MouseBite, F.Cu at (109.2, 92.7)
- added REF**: MouseBite, Custom:MouseBite, F.Cu at (109.2, 91.7)
- added REF**: MouseBite, Custom:MouseBite, F.Cu at (109.2, 90.7)
- added REF**: MouseBite, Custom:MouseBite, F.Cu at (109.2, 89.7)
- added REF**: MouseBite, Custom:MouseBite, F.Cu at (109.2, 124.7)
- added REF**: MouseBite, Custom:MouseBite, F.Cu at (109.2, 88.7)
- added REF**: MouseBite, Custom:MouseBite, F.Cu at (109.2, 87.7)
- added REF**: MouseBite, Custom:MouseBite, F.Cu at (109.2, 86.7)
- added REF**: MouseBite, Custom:MouseBite, F.Cu at (109.2, 85.7)
- added REF**: MouseBite, Custom:MouseBite, F.Cu at (109.2, 84.7)
- added REF**: MouseBite, Custom:MouseBite, F.Cu at (109.2, 83.7)
- added REF**: MouseBite, Custom:MouseBite, F.Cu at (109.2, 82.7)
- added REF**: MouseBite, Custom:MouseBite, F.Cu at (109.2, 81.7)
- added REF**: MouseBite, Custom:MouseBite, F.Cu at (109.2, 80.7)
- added REF**: MouseBite, Custom:MouseBite, F.Cu at (109.2, 79.7)
- added REF**: MouseBite, Custom:MouseBite, F.Cu at (109.2, 123.7)
- added REF**: MouseBite, Custom:MouseBite, F.Cu at (109.2, 78.7)
- added REF**: MouseBite, Custom:MouseBite, F.Cu at (109.2, 77.7)
- added REF**: MouseBite, Custom:MouseBite, F.Cu at (109.2, 76.7)
- added REF**: MouseBite, Custom:MouseBite, F.Cu at (109.2, 75.7)
- added REF**: MouseBite, Custom:MouseBite, F.Cu at (109.2, 74.7)
- added REF**: MouseBite, Custom:MouseBite, F.Cu at (109.2, 73.7)
- added REF**: MouseBite, Custom:MouseBite, F.Cu at (109.2, 72.7)
- added REF**: MouseBite, Custom:MouseBite, F.Cu at (109.2, 71.7)
- added REF**: MouseBite, Custom:MouseBite, F.Cu at (109.2, 70.7)
- added REF**: MouseBite, Custom:MouseBite, F.Cu at (109.2, 69.7)
- added REF**: MouseBite, Custom:MouseBite, F.Cu at (109.2, 122.7)
- added REF**: MouseBite, Custom:MouseBite, F.Cu at (109.2, 68.7)
- added REF**: MouseBite, Custom:MouseBite, F.Cu at (109.2, 67.7)
- added REF**: MouseBite, Custom:MouseBite, F.Cu at (109.2, 66.7)
- added REF**: MouseBite, Custom:MouseBite, F.Cu at (109.2, 121.7)
- added REF**: MouseBite, Custom:MouseBite, F.Cu at (109.2, 120.7)
- added REF**: MouseBite, Custom:MouseBite, F.Cu at (109.2, 119.7)
Other:
- outline, holes or cut-outs redrawn
- board text added: "Max and Chip"
